Commit message: update case2

File: Simulator/gazebo_simulator/turtlebot3_model/urdf/turtlebot3_burger.urdf.xacro (robot description, xacro)
@@ -122,5 +122,5 @@
       <origin xyz="0 0 0.0" rpy="0 0 0"/>
       <geometry>
-        <mesh filename="package://prometheus_gazebo/turtlebot3_model/meshes/sensors/lds.stl" scale="0.001 0.001 0.001"/>
+        <mesh filename="package://prometheus_gazebo/turtlebot3_model/meshes/sensor/lds.stl" scale="0.001 0.001 0.001"/>
       </geometry>
       <material name="dark"/>

File: Simulator/gazebo_simulator/turtlebot3_model/urdf/turtlebot3_waffle.urdf.xacro (robot description, xacro)
@@ -146,5 +146,5 @@
       <origin xyz="0 0 0" rpy="0 0 0"/>
       <geometry>
-        <mesh filename="package://prometheus_gazebo/turtlebot3_model/meshes/sensors/lds.stl" scale="0.001 0.001 0.001"/>
+        <mesh filename="package://prometheus_gazebo/turtlebot3_model/meshes/sensor/lds.stl" scale="0.001 0.001 0.001"/>
       </geometry>
       <material name="dark"/>
@@ -173,5 +173,5 @@
      <origin xyz="0 0 0" rpy="1.57 0 1.57"/>
       <geometry>
-       <mesh filename="package://prometheus_gazebo/turtlebot3_model/meshes/sensors/r200.dae" />
+       <mesh filename="package://prometheus_gazebo/turtlebot3_model/meshes/sensor/r200.dae" />
       </geometry>
     </visual>

File: Simulator/gazebo_simulator/turtlebot3_model/urdf/turtlebot3_waffle_pi.urdf.xacro (robot description, xacro)
@@ -142,5 +142,5 @@
       <origin xyz="0 0 0.0" rpy="0 0 0"/>
       <geometry>
-        <mesh filename="package://prometheus_gazebo/turtlebot3_model/meshes/sensors/lds.stl" scale="0.001 0.001 0.001"/>
+        <mesh filename="package://prometheus_gazebo/turtlebot3_model/meshes/sensor/lds.stl" scale="0.001 0.001 0.001"/>
       </geometry>
       <material name="dark"/>
